File: Nixie.kicad_sch (KiCad schematic)
At the start: 52 parts, among them J1 Led output, J2 Led Input, J3 Conn_01x03, Q1 Q_NMOS_GSD, U1 74LVC1G79, U2 HV5122, U3 HV5122

Commit message: Update PCB layout, schematic, and documentation exports
Parts:
- J1, J2: footprint Connector_PinHeader_1.00mm:PinHeader_1x10_P1.00mm_Vertical -> Connector_PinHeader_1.00mm:PinHeader_1x20_P1.00mm_Vertical
Changed lines of the file:
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@@
 			)
 		)
-		(property "Footprint" "Connector_PinHeader_1.00mm:PinHeader_1x10_P1.00mm_Vertical"
+		(property "Footprint" "Connector_PinHeader_1.00mm:PinHeader_1x20_P1.00mm_Vertical"
 			(at 342.9 64.77 0)
 			(hide yes)
@@
 			)
 		)
-		(property "Footprint" "Connector_PinHeader_1.00mm:PinHeader_1x10_P1.00mm_Vertical"
+		(property "Footprint" "Connector_PinHeader_1.00mm:PinHeader_1x20_P1.00mm_Vertical"
 			(at 312.42 64.77 0)
 			(hide yes)

Commit message: Update schematic connector JP1, PCB routing, BOM, and export files
Parts:
- J1, J2: symbol Connector_Generic:Conn_01x20 -> Connector_Generic:Conn_01x18
- JP1: symbol Connector_Generic:Conn_01x10 -> Connector_Generic:Conn_01x07
Connections:
- net CLK: now also JP1.4 (Pin_4); no longer JP1.7 (Pin_7)
- net DIN: now also JP1.3 (Pin_3); no longer JP1.6 (Pin_6)
- net GND: now also JP1.7 (Pin_7); no longer JP1.10 (Pin_10)
- net OE: now also JP1.5 (Pin_5); no longer JP1.8 (Pin_8)
- net SRB: now also JP1.6 (Pin_6); no longer JP1.9 (Pin_9)
- no-connect marks 10 -> 3

Commit message: Update schematic and export latest schematic PDF
Parts:
- C6, C7, C8, C9: footprint Capacitor_THT:C_Disc_D3.0mm_W2.0mm_P2.50mm -> Capacitor_THT:C_Disc_D4.7mm_W2.5mm_P5.00mm; KiLib_Generator (none) -> capacitor/THT/other
- D5: KiLib_Generator (none) -> LED/THT
- J1, J2: footprint Connector_PinHeader_1.00mm:PinHeader_1x20_P1.00mm_Vertical -> Connector_PinHeader_2.54mm:PinHeader_1x18_P2.54mm_Vertical; KiLib_Generator (none) -> connector/pin_header_socket
- J3: footprint Connector_PinHeader_1.00mm:PinHeader_1x03_P1.00mm_Vertical -> Connector_PinHeader_2.54mm:PinHeader_1x03_P2.54mm_Vertical; KiLib_Generator (none) -> connector/pin_header_socket
- JP1: footprint Connector_PinHeader_1.00mm:PinHeader_1x10_P1.00mm_Vertical -> Connector_PinHeader_2.54mm:PinHeader_1x07_P2.54mm_Vertical; KiLib_Generator (none) -> connector/pin_header_socket
- Q1: KiLib_Generator (none) -> package/gullwing
- R1, R10, R11, R12, R13, R14, R15, R16, R17, R18, R19, R2, R20, R21, R22, R23, R24, R25, R26, R27, R3, R4, R5, R6, R7, R8, R9: KiLib_Generator (none) -> resistor/THT

Commit message: Update design with PLCC-44 IC sockets and SK6812 MINI-E smart RGB LEDs
Parts:
- removed D1, D2, D3, D4, D6, D7: Led_RGB_CA, LED_SMD:LED_Cree-PLCC4_5x5mm_CW, symbol Device:LED_ARGB
- removed J1: Led output, Connector_PinHeader_2.54mm:PinHeader_1x18_P2.54mm_Vertical, symbol Connector_Generic:Conn_01x18
- removed J2: Led Input, Connector_PinHeader_2.54mm:PinHeader_1x18_P2.54mm_Vertical, symbol Connector_Generic:Conn_01x18
- removed J3: Conn_01x03, Connector_PinHeader_2.54mm:PinHeader_1x03_P2.54mm_Vertical, symbol Connector_Generic:Conn_01x03
- removed R10, R13, R16, R20, R23: 100R, Resistor_THT:R_Axial_DIN0207_L6.3mm_D2.5mm_P7.62mm_Horizontal, symbol Device:R
- removed R11, R12, R14, R15, R17, R19, R2, R21, R22, R24, R25, R3: 120R, Resistor_THT:R_Axial_DIN0207_L6.3mm_D2.5mm_P7.62mm_Horizontal, symbol Device:R
- added D1, D2, D3, D4, D6, D7: SK6812MINI-E, LED_SMD:LED_SK6812MINI-E_3.2x2.8mm_P1.5mm_ReverseMount, symbol LED:SK6812MINI-E
- JP1: footprint Connector_PinHeader_2.54mm:PinHeader_1x07_P2.54mm_Vertical -> Connector_PinHeader_2.54mm:PinHeader_1x08_P2.54mm_Vertical; symbol Connector_Generic:Conn_01x07 -> Connector_Generic:Conn_01x08
- R1: value 100R -> 330R; KiLib_Generator resistor/THT -> (none)
Connections:
- net +5V: now also D1.3 (VDD), D2.3 (VDD), D3.3 (VDD), D4.3 (VDD), D6.3 (VDD), D7.3 (VDD)
- net GND: now also D1.1 (VSS), D2.1 (VSS), D3.1 (VSS), D4.1 (VSS), D6.1 (VSS), D7.1 (VSS)
- net LED_DIN: now reaches R1.1
- net LED_DIN: now also D1.2 (DIN)
- net R: no longer names the net of R1.2
- net R: now also JP1.8 (Pin_8)
- new net: D1.4 (DOUT), D2.2 (DIN)
- new net: D2.4 (DOUT), D3.2 (DIN)
- new net: D6.4 (DOUT), D7.2 (DIN)
- new net: D3.4 (DOUT), D4.2 (DIN)
- new net: D4.4 (DOUT), D6.2 (DIN)
- no-connect marks 3 -> 5
